Commit message: mods xacro

File: sr_description/arm/xacro/arm_itself.urdf.xacro (robot description, xacro)
@@ -3,10 +3,15 @@
 xmlns:interface="http://playerstage.sourceforge.net/gazebo/xmlschema/#interface"
 xmlns:xacro="http://www.ros.org/wiki/xacro" name="full_arm_motor">
-  <xacro:include filename="$(find sr_description)/arm/xacro/base/shadowarm_base.urdf.xacro" />
-  <xacro:include filename="$(find sr_description)/arm/xacro/trunk/shadowarm_trunk.urdf.xacro" />
-  <xacro:include filename="$(find sr_description)/arm/xacro/upper_arm/shadowarm_upperarm.urdf.xacro" />
-  <xacro:include filename="$(find sr_description)/arm/xacro/lower_arm/shadowarm_lowerarm.urdf.xacro" />
-  <xacro:include filename="$(find sr_description)/arm/xacro/hand_support/shadowarm_handsupport_motor.urdf.xacro" />
-  <xacro:macro name="sr_arm_motor">
+    <xacro:include filename="$(find sr_description)/arm/xacro/base/shadowarm_base.urdf.xacro" />
+    <xacro:include filename="$(find sr_description)/arm/xacro/trunk/shadowarm_trunk.urdf.xacro" />
+    <xacro:include filename="$(find sr_description)/arm/xacro/upper_arm/shadowarm_upperarm.urdf.xacro" />
+    <xacro:include filename="$(find sr_description)/arm/xacro/lower_arm/shadowarm_lowerarm.urdf.xacro" />
+    <xacro:include filename="$(find sr_description)/arm/xacro/hand_support/shadowarm_handsupport_motor.urdf.xacro" />
+    <link name="world" />
+    <joint name="arm_to_world_fixed" type="fixed">
+        <parent link="world" />
+        <child link="shadowarm_base" />
+        <origin rpy="0 0 0" xyz="0 0 1.0" />
+    </joint>
     <xacro:shadowarm_base></xacro:shadowarm_base>
     <xacro:shadowarm_trunk parent="shadowarm_base">
@@ -18,4 +23,3 @@
     <xacro:shadowarm_handsupport_motor parent="shadowarm_lowerarm">
     </xacro:shadowarm_handsupport_motor>
-  </xacro:macro>
 </robot>

File: sr_description/arm/xacro/base/shadowarm_base.urdf.xacro (robot description, xacro)
@@ -18,13 +18,11 @@
       </visual>
       <collision>
-        <origin xyz="0 0 0.005" rpy="0 0 0" />
-        <geometry name="shadowarm_base_collision">
-          <box size="0.145 0.145 0.012" />
+        <origin xyz="0 0 0" rpy="0 0 0" />
+        <geometry name="shadowarm_base_visual">
+          <mesh filename="package://sr_description/arm/model/arm_base.dae"
+          scale="0.001 0.001 0.001" />
         </geometry>
       </collision>
     </link>
-    <gazebo reference="shadowarm_base">
-      <selfCollide>false</selfCollide>
-    </gazebo>
   </xacro:macro>
 </robot>

File: sr_description/arm/xacro/hand_support/shadowarm_handsupport_motor.urdf.xacro (robot description, xacro)
@@ -1,4 +1,3 @@
 <robot xmlns:xacro="http://www.ros.org/wiki/xacro">
-  <xacro:include filename="$(find sr_description)/arm/xacro/hand_support/shadowarm_handsupport_motor.transmission.xacro" />
   <xacro:macro name="shadowarm_handsupport_motor" params="parent">
     <link name="shadowarm_handsupport">
@@ -18,14 +17,11 @@
       </visual>
       <collision>
-        <origin xyz="0 0 -0.005" rpy="0 0 0" />
-        <geometry name="shadowarm_handsupport_collision">
-          <cylinder radius="0.0675" length="0.006" />
+        <origin xyz="0 0 -0.04" rpy="0 0 0" />
+        <geometry name="shadowarm_handsupport_visual">
+          <mesh filename="package://sr_description/arm/model/elbow_rotate_motor.dae"
+          scale="0.001 0.001 0.001" />
         </geometry>
       </collision>
     </link>
-    <gazebo reference="shadowarm_handsupport">
-      <material>Gazebo/Grey</material>
-      <selfCollide>false</selfCollide>
-    </gazebo>
     <joint name="ElbowJRotate" type="revolute">
       <parent link="${parent}" />
@@ -37,9 +33,4 @@
       <dynamics damping="5.5" />
     </joint>
-    <gazebo reference="ElbowJRotate">
-      <provideFeedback>1</provideFeedback>
-      <implicitSpringDamper>1</implicitSpringDamper>
-    </gazebo>
-    <xacro:shadowarm_handsupport_motor_transmission />
   </xacro:macro>
 </robot>

File: sr_description/arm/xacro/lower_arm/shadowarm_lowerarm.urdf.xacro (robot description, xacro)
@@ -1,4 +1,3 @@
 <robot xmlns:xacro="http://www.ros.org/wiki/xacro">
-  <xacro:include filename="$(find sr_description)/arm/xacro/lower_arm/shadowarm_lowerarm.transmission.xacro" />
   <xacro:macro name="shadowarm_lowerarm" params="parent">
     <link name="shadowarm_lowerarm">
@@ -18,13 +17,11 @@
       </visual>
       <collision>
-        <origin xyz="0.08 0 0.0625" rpy="0 0 0" />
-        <geometry name="shadowarm_lowerarm_collision">
-          <box size="0.06 0.08 0.1" />
+        <origin xyz="0.03 0 0.036" rpy="0 0 0" />
+        <geometry name="shadowarm_lowerarm_visual">
+          <mesh filename="package://sr_description/arm/model/elbow_flex.dae"
+          scale="0.001 0.001 0.001" />
         </geometry>
       </collision>
     </link>
-    <gazebo reference="shadowarm_lowerarm">
-      <selfCollide>false</selfCollide>
-    </gazebo>
     <joint name="ElbowJSwing" type="revolute">
       <parent link="${parent}" />
@@ -36,9 +33,4 @@
       <dynamics damping="5.5" />
     </joint>
-    <gazebo reference="ElbowJSwing">
-      <provideFeedback>1</provideFeedback>
-      <implicitSpringDamper>1</implicitSpringDamper>
-    </gazebo>
-    <xacro:shadowarm_lowerarm_transmission />
   </xacro:macro>
 </robot>

File: sr_description/arm/xacro/trunk/shadowarm_trunk.urdf.xacro (robot description, xacro)
@@ -1,4 +1,3 @@
 <robot xmlns:xacro="http://www.ros.org/wiki/xacro">
-  <xacro:include filename="$(find sr_description)/arm/xacro/trunk/shadowarm_trunk.transmission.xacro" />
   <xacro:macro name="shadowarm_trunk" params="parent">
     <link name="shadowarm_trunk">
@@ -18,13 +17,11 @@
       </visual>
       <collision>
-        <origin xyz="0 0.02 0.30" rpy="0 0 0" />
-        <geometry name="shadowarm_trunk_collision">
-          <box size="0.170 0.170 0.580" />
+        <origin xyz="0 0 0.005" rpy="0 0 0" />
+        <geometry name="shadowarm_trunk_visual">
+          <mesh filename="package://sr_description/arm/model/arm_trunk.dae"
+          scale="0.001 0.001 0.001" />
         </geometry>
       </collision>
     </link>
-    <gazebo reference="shadowarm_trunk">
-      <selfCollide>false</selfCollide>
-    </gazebo>
     <joint name="ShoulderJRotate" type="revolute">
       <parent link="${parent}" />
@@ -36,9 +33,4 @@
       <dynamics damping="5.5" />
     </joint>
-    <gazebo reference="ShoulderJRotate">
-      <provideFeedback>1</provideFeedback>
-      <implicitSpringDamper>1</implicitSpringDamper>
-    </gazebo>
-    <xacro:shadowarm_trunk_transmission />
   </xacro:macro>
 </robot>

File: sr_description/arm/xacro/upper_arm/shadowarm_upperarm.urdf.xacro (robot description, xacro)
@@ -1,4 +1,3 @@
 <robot xmlns:xacro="http://www.ros.org/wiki/xacro">
-  <xacro:include filename="$(find sr_description)/arm/xacro/upper_arm/shadowarm_upperarm.transmission.xacro" />
   <xacro:macro name="shadowarm_upperarm" params="parent">
     <link name="shadowarm_upperarm">
@@ -18,13 +17,11 @@
       </visual>
       <collision>
-        <origin xyz="0 0 0.16" rpy="0 -${M_PI} 0" />
-        <geometry name="shadowarm_upperarm_collision">
-          <box size="0.170 0.133 0.470" />
+        <origin xyz="0 0.067 0" rpy="0 0 0" />
+        <geometry name="shadowarm_upperarm_visual">
+          <mesh filename="package://sr_description/arm/model/upper_arm.dae"
+          scale="0.001 0.001 0.001" />
         </geometry>
       </collision>
     </link>
-    <gazebo reference="shadowarm_upperarm">
-      <selfCollide>false</selfCollide>
-    </gazebo>
     <joint name="ShoulderJSwing" type="revolute">
       <parent link="${parent}" />
@@ -37,9 +34,4 @@
       <dynamics damping="5.3" />
     </joint>
-    <gazebo reference="ShoulderJSwing">
-      <provideFeedback>1</provideFeedback>
-      <implicitSpringDamper>1</implicitSpringDamper>
-    </gazebo>
-    <xacro:shadowarm_upperarm_transmission />
   </xacro:macro>
 </robot>
