Commit message: delete forearm urdf

File: sr_description/robots/shadowhand_motor.urdf (robot description, URDF)
Before this commit: robot shadowhand_motor, 33 links, 32 joints
Links:
- removed link rh_forearm
- removed link rh_imu
- removed link rh_manipulator
- removed link rh_wrist
- removed link world
Joints:
- removed joint rh_WRJ1
- removed joint rh_WRJ2
- removed joint rh_ee_fixed_joint
- removed joint rh_palm_to_imu
- removed joint rh_world_joint
