Commit message: add wrist jl back

File: sr_description/robots/shadowhand_motor_simple_nomass.urdf (robot description, URDF)
Before this commit: robot shadowhand_motor, 30 links, 29 joints
Joints:
- joint world_rx: limit lower=-1000 upper=1000 effort=10000.0 velocity=1000.0 -> lower=-0.7 upper=0.7 effort=10000.0 velocity=1000.0
- joint world_ry: limit lower=-1000 upper=1000 effort=10000.0 velocity=1000.0 -> lower=-0.7 upper=0.7 effort=10000.0 velocity=1000.0
- joint world_rz: limit lower=-1000 upper=1000 effort=10000.0 velocity=1000.0 -> lower=-0.7 upper=0.7 effort=10000.0 velocity=1000.0
- joint world_x: limit lower=-1000 upper=1000 effort=10000.0 velocity=1000.0 -> lower=-0.1 upper=0.2 effort=10000.0 velocity=1000.0
- joint world_y: limit lower=-1000 upper=1000 effort=10000.0 velocity=1000.0 -> lower=-0.1 upper=0.1 effort=10000.0 velocity=1000.0
- joint world_z: limit lower=-1000 upper=1000 effort=10000.0 velocity=1000.0 -> lower=-0.1 upper=0.1 effort=10000.0 velocity=1000.0

Commit message: lock wrist -x

File: sr_description/robots/shadowhand_motor_simple_nomass.urdf (robot description, URDF)
Before this commit: robot shadowhand_motor, 30 links, 29 joints
Joints:
- joint world_x: limit lower=-0.1 upper=0.2 effort=10000.0 velocity=1000.0 -> lower=-0.01 upper=0.35 effort=10000.0 velocity=1000.0
