Commit message: remove forearm for inmoov

File: sr_description/hand/xacro/full_hand.urdf.xacro (robot description, xacro)
@@ -19,8 +19,8 @@
   <!-- lf is true if we want a little finger, false otherwise -->
   <xacro:macro name="shadowhand"
-  params="muscletrans muscle hand_type:='hand_e' bio bt_sp ubi eli reflect prefix lf cable_mesh:='false'">
+  params="muscletrans muscle hand_type:='hand_e' bio bt_sp ubi eli reflect prefix lf cable_mesh:='false' parent">
     <!--xacro:property name="hand_type" value="hand_e"/-->
     <!-- Forearm -->
-    <xacro:forearm muscle="${muscle}" hand_type="${hand_type}" prefix="${prefix}" cable_mesh="${cable_mesh}"/>
+    <!-- <xacro:forearm muscle="${muscle}" hand_type="${hand_type}" prefix="${prefix}" cable_mesh="${cable_mesh}"/> -->
     <!-- Wrist -->
     <xacro:if value="${muscle}">
@@ -32,6 +32,6 @@
     <xacro:unless value="${muscle}">
       <xacro:wrist muscletrans="false" prefix="${prefix}"
-      reflect="${reflect}" parent="${prefix}forearm">
-        <origin xyz="0 -0.010 0.213" rpy="0 0 0" />
+      reflect="${reflect}" parent="${parent}">
+        <origin xyz="0 -0.010 0.0" rpy="0 0 0" />
       </xacro:wrist>
     </xacro:unless>

File: sr_description/hand/xacro/palm/palm.urdf.xacro (robot description, xacro)
@@ -108,5 +108,5 @@
     </gazebo>
     <!--imu-->
-    <xacro:imu prefix="${prefix}"/>
+    <!-- <xacro:imu prefix="${prefix}"/> -->
     <!-- extensions -->
     <xacro:shadowhand_palm_transmission muscletrans="${muscletrans}"

File: sr_description/robots/shadowhand_motor.urdf.xacro (robot description, xacro)
@@ -9,10 +9,10 @@
     <!-- hand with cylindrical base drifts in gazebo, attach it to the world -->
     <link name="world" />
-    <joint name="rh_world_joint" type="fixed">
+    <!-- <joint name="rh_world_joint" type="fixed">
       <parent link="world" />
       <child link="rh_forearm" />
       <origin xyz="0.0 0.0 0.0" rpy="0.0 0.0 0.0" />
-    </joint>
+    </joint> -->
     <xacro:shadowhand muscletrans="false" muscle="false" hand_type="hand_e" bio="false" bt_sp="false"
-                      ubi="false" eli="false" reflect="1.0" prefix="rh_" lf="true" />
+                      ubi="false" eli="false" reflect="1.0" prefix="rh_" lf="true" parent="world"/>
 </robot>

Commit message: more mods for inmoov

File: sr_description/hand/xacro/full_hand.urdf.xacro (robot description, xacro)
@@ -3,5 +3,5 @@
 xmlns:interface="http://playerstage.sourceforge.net/gazebo/xmlschema/#interface"
 xmlns:xacro="http://www.ros.org/wiki/xacro">
-  <xacro:include filename="$(find sr_description)/hand/xacro/forearm/forearm.urdf.xacro" />
+  <!-- <xacro:include filename="$(find sr_description)/hand/xacro/forearm/forearm.urdf.xacro" /> -->
   <xacro:include filename="$(find sr_description)/hand/xacro/wrist/wrist.urdf.xacro" />
   <xacro:include filename="$(find sr_description)/hand/xacro/palm/palm.urdf.xacro" />
@@ -26,5 +26,5 @@
     <xacro:if value="${muscle}">
       <xacro:wrist muscletrans="${muscletrans}" prefix="${prefix}"
-      reflect="${reflect}" parent="${prefix}forearm">
+      reflect="${reflect}" parent="${parent}">
         <origin xyz="0 0 0.4096" rpy="0 0 0" />
       </xacro:wrist>
@@ -33,5 +33,5 @@
       <xacro:wrist muscletrans="false" prefix="${prefix}"
       reflect="${reflect}" parent="${parent}">
-        <origin xyz="0 -0.010 0.0" rpy="0 0 0" />
+        <origin xyz="0 0.0 0.0" rpy="0 0 0" />
       </xacro:wrist>
     </xacro:unless>

File: sr_description/hand/xacro/palm/palm.urdf.xacro (robot description, xacro)
@@ -97,8 +97,9 @@
       <parent link="${parent}" />
       <child link="${prefix}palm" />
-      <origin xyz="0 0 0.034" rpy="0 0 0" />
+      <origin xyz="0 0 0.03" rpy="0 0 0" />
       <axis xyz="1 0 0" />
-      <limit lower="${-40/180*M_PI}" upper="${28/180*M_PI}"
-      effort="30" velocity="2.0" />
+      <!-- this is the wrist flexion -->
+      <limit lower="${-90/180*M_PI}" upper="${90/180*M_PI}"
+      effort="30" velocity="20.0" />
       <dynamics damping="0.1" />
     </joint>

File: sr_description/hand/xacro/wrist/wrist.urdf.xacro (robot description, xacro)
@@ -63,7 +63,8 @@
       <child link="${prefix}wrist" />
       <xacro:insert_block name="origin" />
+      <!-- this is the wrist adduction -->
       <axis xyz="0 ${reflect} 0" />
-      <limit lower="${-30/180*M_PI}" upper="${10/180*M_PI}"
-      effort="10" velocity="2.0" />
+      <limit lower="${-60/180*M_PI}" upper="${60/180*M_PI}"
+      effort="10" velocity="20.0" />
       <dynamics damping="0.1" />
     </joint>

Commit message: match xacro to urdf neither have unused link

File: sr_description/hand/xacro/full_hand.urdf.xacro (robot description, xacro)
@@ -19,24 +19,31 @@
   <!-- lf is true if we want a little finger, false otherwise -->
   <xacro:macro name="shadowhand"
-  params="muscletrans muscle hand_type:='hand_e' bio bt_sp ubi eli reflect prefix lf cable_mesh:='false' parent">
+  params="muscletrans muscle hand_type:='hand_e' bio bt_sp ubi eli reflect prefix lf cable_mesh:='false' parent no_arm:='false'">
     <!--xacro:property name="hand_type" value="hand_e"/-->
     <!-- Forearm -->
     <!-- <xacro:forearm muscle="${muscle}" hand_type="${hand_type}" prefix="${prefix}" cable_mesh="${cable_mesh}"/> -->
-    <!-- Wrist -->
-    <xacro:if value="${muscle}">
-      <xacro:wrist muscletrans="${muscletrans}" prefix="${prefix}"
-      reflect="${reflect}" parent="${parent}">
-        <origin xyz="0 0 0.4096" rpy="0 0 0" />
-      </xacro:wrist>
+    <xacro:if value="${no_arm}">
+      <!-- Palm -->
+      <xacro:palm muscletrans="${muscletrans}" prefix="${prefix}"
+      reflect="${reflect}" is_root="true" parent="dummy"/>
     </xacro:if>
-    <xacro:unless value="${muscle}">
-      <xacro:wrist muscletrans="false" prefix="${prefix}"
-      reflect="${reflect}" parent="${parent}">
-        <origin xyz="0 0.0 0.0" rpy="0 0 0" />
-      </xacro:wrist>
+    <xacro:unless value="${no_arm}">
+      <!-- Wrist -->
+      <xacro:if value="${muscle}">
+        <xacro:wrist muscletrans="${muscletrans}" prefix="${prefix}"
+        reflect="${reflect}" parent="${parent}">
+          <origin xyz="0 0 0.4096" rpy="0 0 0" />
+        </xacro:wrist>
+      </xacro:if>
+      <xacro:unless value="${muscle}">
+        <xacro:wrist muscletrans="false" prefix="${prefix}"
+        reflect="${reflect}" parent="${parent}">
+          <origin xyz="0 0.0 0.0" rpy="0 0 0" />
+        </xacro:wrist>
+      </xacro:unless>
+      <!-- Palm -->
+      <xacro:palm muscletrans="${muscletrans}" prefix="${prefix}"
+      reflect="${reflect}" parent="${prefix}wrist" />
     </xacro:unless>
-    <!-- Palm -->
-    <xacro:palm muscletrans="${muscletrans}" prefix="${prefix}"
-    reflect="${reflect}" parent="${prefix}wrist" />
     <!-- First Finger -->
     <xacro:finger muscletrans="${muscletrans}" lf="false"

File: sr_description/hand/xacro/palm/palm.urdf.xacro (robot description, xacro)
@@ -14,5 +14,5 @@
   <!-- parent is the parent link for the joint -->
   <xacro:macro name="palm"
-  params="muscletrans prefix reflect parent">
+  params="muscletrans prefix reflect is_root:='false' parent">
     <link name="${prefix}palm">
       <inertial>
@@ -88,29 +88,29 @@
       </collision>
     </link>
-    <joint name="${prefix}ee_fixed_joint" type="fixed">
+    <!-- <joint name="${prefix}ee_fixed_joint" type="fixed">
       <parent link="${prefix}palm" />
       <child link = "${prefix}manipulator" />
       <origin xyz="0.0 0.0 0.05" rpy="0.0 0.0 0.0" />
     </joint>
-    <link name="${prefix}manipulator" />
-    <joint name="${prefix}WRJ1" type="revolute">
-      <parent link="${parent}" />
-      <child link="${prefix}palm" />
-      <origin xyz="0 0 0.03" rpy="0 0 0" />
-      <axis xyz="1 0 0" />
-      <!-- this is the wrist flexion -->
-      <limit lower="${-90/180*M_PI}" upper="${90/180*M_PI}"
-      effort="30" velocity="20.0" />
-      <dynamics damping="0.1" />
-    </joint>
-    <gazebo reference="${prefix}WRJ1">
-      <provideFeedback>1</provideFeedback>
-      <implicitSpringDamper>1</implicitSpringDamper>
-    </gazebo>
+    <link name="${prefix}manipulator" /> -->
+    <xacro:unless value="${is_root}">
+      <joint name="${prefix}WRJ1" type="revolute">
+        <parent link="${parent}" />
+        <child link="${prefix}palm" />
+        <origin xyz="0 0 0.03" rpy="0 0 0" />
+        <axis xyz="1 0 0" />
+        <!-- this is the wrist flexion -->
+        <limit lower="${-90/180*M_PI}" upper="${90/180*M_PI}"
+        effort="30" velocity="20.0" />
+        <dynamics damping="0.1" />
+      </joint>
+      <gazebo reference="${prefix}WRJ1">
+        <provideFeedback>1</provideFeedback>
+        <implicitSpringDamper>1</implicitSpringDamper>
+      </gazebo>
+    </xacro:unless>
     <!--imu-->
     <!-- <xacro:imu prefix="${prefix}"/> -->
     <!-- extensions -->
-    <xacro:shadowhand_palm_transmission muscletrans="${muscletrans}"
-    prefix="${prefix}" />
     <xacro:shadowhand_palm_gazebo prefix="${prefix}" />
   </xacro:macro>

File: sr_description/robots/shadowhand_motor.urdf.xacro (robot description, xacro)
@@ -8,5 +8,5 @@
     <xacro:include filename="$(find sr_description)/other/xacro/gazebo/gazebo.urdf.xacro"/>
     <!-- hand with cylindrical base drifts in gazebo, attach it to the world -->
-    <link name="world" />
+    <!-- <link name="world" /> -->
     <!-- <joint name="rh_world_joint" type="fixed">
       <parent link="world" />
@@ -15,4 +15,4 @@
     </joint> -->
     <xacro:shadowhand muscletrans="false" muscle="false" hand_type="hand_e" bio="false" bt_sp="false"
-                      ubi="false" eli="false" reflect="1.0" prefix="rh_" lf="true" parent="world"/>
+                      ubi="false" eli="false" reflect="1.0" prefix="rh_" lf="true" parent="world" no_arm="true"/>
 </robot>
