Commit message: add palm_aux

File: sr_description/hand/xacro/palm/palm.urdf.xacro (robot description, xacro)
@@ -15,4 +15,11 @@
   <xacro:macro name="palm"
   params="muscletrans prefix reflect is_root:='false' parent">
+    <link name="${prefix}palm_aux">
+      <inertial>
+        <origin rpy="0 0 0" xyz="0 0 0"/>
+        <mass value="0.003"/>
+        <inertia ixx="0.00001" ixy="0" ixz="0" iyy="0.00001" iyz="0" izz="0.00001"/>
+      </inertial>
+    </link>
     <link name="${prefix}palm">
       <inertial>
@@ -97,5 +104,5 @@
       <joint name="${prefix}WRJ1" type="revolute">
         <parent link="${parent}" />
-        <child link="${prefix}palm" />
+        <child link="${prefix}palm_aux" />
         <origin xyz="0 0 0.03" rpy="0 0 0" />
         <axis xyz="1 0 0" />
@@ -110,4 +117,9 @@
       </gazebo>
     </xacro:unless>
+    <joint name="${prefix}palm_aux_joint" type="fixed">
+      <origin rpy="0 0 0" xyz="0 0.0 0.0"/>
+      <parent link="${prefix}palm_aux"/>
+      <child link="${prefix}palm"/>
+    </joint>
     <!--imu-->
     <!-- <xacro:imu prefix="${prefix}"/> -->

File: sr_description/robots/shadowhand_motor.urdf (robot description, URDF)
Before this commit: robot shadowhand_motor, 28 links, 27 joints
Links:
- added link rh_palm_aux, mass 0.003
Joints:
- added joint rh_palm_aux_joint: type fixed, parent rh_palm_aux, child rh_palm, origin xyz=0 0.0 0.0 rpy=0 0 0
